Commit message: modified

File: realsense2_camera/urdf/test_d435_camera.urdf.sim.xacro (robot description, xacro)
@@ -1,13 +1,9 @@
 <?xml version="1.0"?>
 <robot name="realsense2_camera" xmlns:xacro="http://ros.org/wiki/xacro">
-  <xacro:include filename="$(find realsense2_camera)/urdf/_d435.urdf.xacro"/>
-  <sensor_d435 parent="tools2">
-    <origin xyz="-0.01 -0.435 0.015" rpy="1.5707963 0 3.1415926"/>
-  </sensor_d435>
   <link
     name="tools1">
     <inertial>
       <origin
-        xyz="0 -0.5 0"
+        xyz="0 0 0"
         rpy="0 0 0" />
       <mass
@@ -23,5 +19,5 @@
     <visual>
       <origin
-        xyz="0 -0.5 0"
+        xyz="0 0 0.5"
         rpy="0 0 0" />
       <geometry>
@@ -37,7 +33,7 @@
       </material>
     </visual>
-    <collision>
+    <!--collision>
       <origin
-        xyz="0 -0.5 0"
+        xyz="0 0 0"
         rpy="0 0 0" />
       <geometry>
@@ -45,5 +41,5 @@
           filename="$(find kinova_description)/objects/tools/first.dae" />
       </geometry>
-    </collision>
+    </collision>-->
   </link>
   <joint
@@ -51,6 +47,6 @@
     type="fixed">
     <origin
-      xyz="-0.0323 -0.040 -0.5"
-      rpy="-1.5707963 0 0" />
+      xyz="0 0 0.5"
+      rpy="0 0 0" />
     <parent
       link="j2s7s300_link_7" />
@@ -60,61 +56,3 @@
       xyz="0 0 0" />
   </joint>
-<link
-    name="tools2">
-    <inertial>
-      <origin
-        xyz="0 -0.5 0"
-        rpy="0 0 0" />
-      <mass
-        value="2.0243E-6" />
-      <inertia
-        ixx="0.031947E-6"
-        ixy="-6.6313E-24"
-        ixz="-2.4676E-24"
-        iyy="0.023762E-6"
-        iyz="-7.8627E-24"
-        izz="0.052372E-6" />
-    </inertial>
-    <visual>
-      <origin
-        xyz="0 -0.5 0"
-        rpy="0 0 0" />
-      <geometry>
-        <mesh
-          filename="$(find kinova_description)/objects/tools/second.dae" />
-      </geometry>
-      <material
-        name="">
-        <color
-          rgba="1 1 1 1" />
-        <texture
-          filename="$(find kinova_description)/objects//textures/blue.jpg" />
-      </material>
-    </visual>
-    <collision>
-      <origin
-        xyz="0 -0.5 0"
-        rpy="0 0 0" />
-      <geometry>
-        <mesh
-          filename="$(find kinova_description)/objects/tools/second.dae" />
-      </geometry>
-    </collision>
-    <gazebo >
-      <material>Gazebo/blue</material>
-    </gazebo>
-</link>
-  <joint
-    name="joint_tools2"
-    type="fixed">
-    <origin
-      xyz="0.016 -0.5 -0.48"
-      rpy="-1.5707963 0 -1.5707963" />
-    <parent
-      link="tools1" />
-    <child
-      link="tools2" />
-    <axis
-      xyz="0 0 0" />
-  </joint>
 </robot>
